File: pcb/babycounter.kicad_pcb (KiCad board)
At the start: 4 copper layers, 17 parts, among them J1 Conn_01x04_Pin, J2 Conn_01x02_Pin, J3 Conn_01x04_Pin, J4 Conn_01x04_Pin, U1 ESP32-C3_SUPERMINI_SMD, U2 MAX7219, U3 LM317_TO-220

Commit message: 1.5v traces
Connections:
- U2 pad 10: Net-(J3-Pin_4) -> Net-(J3-Pin_2)
- U2 pad 5: Net-(J3-Pin_3) -> Net-(J3-Pin_4)
- U2 pad 8: Net-(J3-Pin_2) -> Net-(J3-Pin_3)
Routing:
- net GND: track 81.8 -> 153.7 mm
- net /1.5V: track 0.00 -> 63.2 mm
- net Net-(U3-ADJ): track 0.00 -> 43.3 mm
- net Net-(DS1-G): track 118.5 -> 156.6 mm
- net Net-(J3-Pin_2): track 0.00 -> 32.0 mm
- net Net-(J3-Pin_3): track 0.00 -> 25.9 mm
- net Net-(J3-Pin_4): track 0.00 -> 18.6 mm
- net Net-(U2-DIG_0): track 0.00 -> 12.1 mm
- net Net-(J3-Pin_1): track 0.00 -> 7.18 mm
Changed lines of the file:
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@@
 		)
 		(property "Value" "D1X8K-14BL"
-			(at 22.735714 20.32 -0)
+			(at 22.735714 20.32 0)
 			(unlocked yes)
 			(layer "B.Fab")
@@
 		)
 		(property "Value" "D1X8K-14BL"
-			(at -27.264286 20.32 -0)
+			(at -27.264286 20.32 0)
 			(unlocked yes)
 			(layer "B.Fab")
@@
 			(layers "*.Cu" "*.Mask")
 			(remove_unused_layers no)
-			(net 22 "Net-(J3-Pin_3)")
+			(net 23 "Net-(J3-Pin_4)")
 			(pinfunction "DIG_6")
 			(pintype "output")
@@
 			(layers "*.Cu" "*.Mask")
 			(remove_unused_layers no)
-			(net 21 "Net-(J3-Pin_2)")
+			(net 22 "Net-(J3-Pin_3)")
 			(pinfunction "DIG_7")
 			(pintype "output")
@@
 			(layers "*.Cu" "*.Mask")
 			(remove_unused_layers no)
-			(net 23 "Net-(J3-Pin_4)")
+			(net 21 "Net-(J3-Pin_2)")
 			(pinfunction "DIG_5")
 			(pintype "output")
@@
 	)
 	(segment
+		(start 168.611277 83.111277)
+		(end 174 88.5)
+		(width 1)
+		(layer "In1.Cu")
+		(net 1)
+	)
+	(segment
+		(start 106.421392 83.111277)
+		(end 168.611277 83.111277)
+		(width 1)
+		(layer "In1.Cu")
+		(net 1)
+	)
+	(segment
 		(start 104.920392 81.420392)
 		(end 104.920392 84.612277)
@@
 	)
 	(segment
+		(start 104.920392 84.612277)
+		(end 106.421392 83.111277)
+		(width 1)
+		(layer "In1.Cu")
+		(net 1)
+	)
+	(segment
 		(start 193.949 81.551)
 		(end 193.949 93.449)
@@
 	)
 	(segment
+		(start 82.5 89.5)
+		(end 81 88)
+		(width 0.5)
+		(layer "F.Cu")
+		(net 4)
+	)
+	(segment
 		(start 156 71.499)
 		(end 156 73)
@@
 	)
 	(segment
+		(start 81 88)
+		(end 81 73)
+		(width 0.5)
+		(layer "F.Cu")
+		(net 4)
+	)
+	(segment
+		(start 102.380392 92.232277)
+		(end 99.648115 89.5)
+		(width 0.5)
+		(layer "F.Cu")
+		(net 4)
+	)
+	(segment
+		(start 99.648115 89.5)
+		(end 82.5 89.5)
+		(width 0.5)
+		(layer "F.Cu")
+		(net 4)
+	)
+	(segment
 		(start 81 73)
 		(end 82.501 71.499)
@@
 	)
 	(segment
+		(start 87.140392 79.140392)
+		(end 87.140392 84.612277)
+		(width 0.5)
+		(layer "B.Cu")
+		(net 6)
+	)
+	(segment
+		(start 86.08 78.08)
+		(end 87.140392 79.140392)
+		(width 0.5)
+		(layer "B.Cu")
+		(net 6)
+	)
+	(segment
+		(start 86.08 73)
+		(end 86.08 78.08)
+		(width 0.5)
+		(layer "B.Cu")
+		(net 6)
+	)
+	(segment
 		(start 138.62 104.88)
 		(end 138.62 103.48)
@@
 	)
 	(segment
+		(start 136 98.855)
+		(end 138.145 101)
+		(width 0.5)
+		(layer "F.Cu")
+		(net 19)
+	)
+	(segment
+		(start 136 97.45)
+		(end 136 98.855)
+		(width 0.5)
+		(layer "F.Cu")
+		(net 19)
+	)
+	(segment
+		(start 138.145 101)
+		(end 187.58 101)
+		(width 0.5)
+		(layer "F.Cu")
+		(net 19)
+	)
+	(segment
+		(start 187.58 101)
+		(end 190.08 98.5)
+		(width 0.5)
+		(layer "F.Cu")
+		(net 19)
+	)
+	(segment
+		(start 194.54 98.5)
+		(end 195.5 97.54)
+		(width 0.5)
+		(layer "B.Cu")
+		(net 19)
+	)
+	(segment
+		(start 190.08 98.5)
+		(end 194.54 98.5)
+		(width 0.5)
+		(layer "B.Cu")
+		(net 19)
+	)
+	(segment
+		(start 84.600392 92.232277)
+		(end 77.692277 92.232277)
+		(width 0.5)
+		(layer "B.Cu")
+		(net 20)
+	)
+	(segment
+		(start 77.692277 92.232277)
+		(end 77.5 92.04)
+		(width 0.5)
+		(layer "B.Cu")
+		(net 20)
+	)
+	(segment
+		(start 79.451 87.549)
+		(end 104.523669 87.549)
+		(width 0.5)
+		(layer "B.Cu")
+		(net 21)
+	)
+	(segment
+		(start 77.5 89.5)
+		(end 79.451 87.549)
+		(width 0.5)
+		(layer "B.Cu")
+		(net 21)
+	)
+	(segment
+		(start 104.523669 87.549)
+		(end 107.460392 84.612277)
+		(width 0.5)
+		(layer "B.Cu")
+		(net 21)
+	)
+	(segment
+		(start 77.612 86.848)
+		(end 77.5 86.96)
+		(width 0.5)
+		(layer "B.Cu")
+		(net 22)
+	)
+	(segment
+		(start 102.380392 84.612277)
+		(end 100.144669 86.848)
+		(width 0.5)
+		(layer "B.Cu")
+		(net 22)
+	)
+	(segment
+		(start 77.5 86.96)
+		(end 77.54 87)
+		(width 0.5)
+		(layer "B.Cu")
+		(net 22)
+	)
+	(segment
+		(start 100.144669 86.848)
+		(end 77.612 86.848)
+		(width 0.5)
+		(layer "B.Cu")
+		(net 22)
+	)
+	(segment
+		(start 79.227 86.147)
+		(end 93.225669 86.147)
+		(width 0.5)
+		(layer "B.Cu")
+		(net 23)
+	)
+	(segment
+		(start 77.5 84.42)
+		(end 79.227 86.147)
+		(width 0.5)
+		(layer "B.Cu")
+		(net 23)
+	)
+	(segment
+		(start 93.225669 86.147)
+		(end 94.760392 84.612277)
+		(width 0.5)
+		(layer "B.Cu")
+		(net 23)
+	)
+	(segment
 		(start 99.840392 93.180392)
 		(end 99.840392 92.232277)
@@
 		(net 28)
 	)
+	(segment
+		(start 175.281 100.299)
+		(end 177.08 98.5)
+		(width 0.5)
+		(layer "F.Cu")
+		(net 29)
+	)
+	(segment
+		(start 141.389 100.299)
+		(end 175.281 100.299)
+		(width 0.5)
+		(layer "F.Cu")
+		(net 29)
+	)
+	(segment
+		(start 138.54 97.45)
+		(end 141.389 100.299)
+		(width 0.5)
+		(layer "F.Cu")
+		(net 29)
+	)
+	(segment
+		(start 177.08 98.5)
+		(end 179.92 98.5)
+		(width 0.5)
+		(layer "B.Cu")
+		(net 29)
+	)
 	(embedded_fonts no)

Commit message: pcb done
Parts:
- moved J4 4.57 mm to (155.0, 94.0)
Routing:
- net Net-(U2-DIG_4): track 0.00 -> 153.5 mm, vias 0 -> 3
- net Net-(U2-DIG_2): track 0.00 -> 104.7 mm, vias 0 -> 7
- net Net-(U2-DIG_3): track 0.00 -> 94.1 mm, vias 0 -> 5
- net Net-(U1-GPIO5): track 0.00 -> 91.9 mm, vias 0 -> 1
- net Net-(U1-GPIO4): track 0.00 -> 84.2 mm
- net Net-(U1-GPIO10): track 0.00 -> 76.0 mm
- net Net-(U2-V+): track 94.3 -> 140.2 mm, vias 0 -> 1
- net Net-(DS1-B): track 118.8 -> 162.0 mm, vias 0 -> 4
- net Net-(U2-DIG_1): track 0.00 -> 41.0 mm, vias 0 -> 5
- net Net-(J4-Pin_3): track 0.00 -> 36.6 mm, vias 0 -> 1
- net Net-(J4-Pin_1): track 0.00 -> 34.8 mm, vias 0 -> 1
- net Net-(U2-DIG_0): track 12.1 -> 46.7 mm, vias 0 -> 2
- net Net-(DS1-C): track 118.7 -> 153.1 mm
- net Net-(J4-Pin_4): track 0.00 -> 32.0 mm, vias 0 -> 1
- net Net-(DS1-F): track 119.0 -> 148.7 mm
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Other:
- board outline added: 126 x 36.5 mm
- copper layers 4 -> 2

Commit message: full plane
Routing:
- net GND: track 160.5 -> 191.5 mm, vias 3 -> 29
- net Net-(U2-DIG_2): track 104.7 -> 105.6 mm
- added copper zone on B.Cu, net GND
- added copper zone on F.Cu, net GND

Commit message: finished board
Routing:
- net Net-(DS1-A): track 143.1 -> 156.8 mm
Other:
- board text added: "DOUT / D5 / D7 / D6"
- board text added: "ESP GPIO 20 / 21 / 6 / 1"
- board text added: "GND 1.5V"
- board text added: "GND 3.3V GPIO 0 GPIO 3"
- board text added: "Made by Hannes :)"
Changed lines of the file:
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@@
 			(outputformat 1)
 			(mirror no)
-			(drillshape 1)
+			(drillshape 0)
 			(scaleselection 1)
-			(outputdirectory "")
+			(outputdirectory "output/")
 		)
 	)
@@
 		(layer "Edge.Cuts")
 	)
+	(gr_text "GND\n1.5V"
+		(at 197 102 0)
+		(layer "B.SilkS")
+		(effects
+			(font
+				(size 1 1)
+				(thickness 0.1)
+			)
+			(justify left bottom mirror)
+		)
+	)
+	(gr_text "ESP GPIO\n20 / 21 / 6 / 1"
+		(at 159.5 92 0)
+		(layer "B.SilkS")
+		(effects
+			(font
+				(size 1 1)
+				(thickness 0.1)
+			)
+			(justify bottom mirror)
+		)
+	)
+	(gr_text "DOUT / D5 / D7 / D6"
+		(at 74 97 270)
+		(layer "B.SilkS")
+		(effects
+			(font
+				(size 1 1)
+				(thickness 0.1)
+			)
+			(justify left bottom mirror)
+		)
+	)
+	(gr_text "GND\n3.3V\nGPIO 0\nGPIO 3"
+		(at 198 77 0)
+		(layer "B.SilkS")
+		(effects
+			(font
+				(size 1 1)
+				(thickness 0.1)
+			)
+			(justify left bottom mirror)
+		)
+	)
+	(gr_text "Made by Hannes :)"
+		(at 133.5 81.5 -0)
+		(layer "B.SilkS")
+		(effects
+			(font
+				(size 1 1)
+				(thickness 0.1)
+			)
+			(justify left bottom mirror)
+		)
+	)
 	(segment
 		(start 93.705113 79.5)
@@
 	)
 	(segment
+		(start 163.5 71.499)
+		(end 163.62 71.619)
+		(width 1)
+		(layer "B.Cu")
+		(net 8)
+	)
+	(segment
+		(start 113.62 71.619)
+		(end 113.5 71.499)
+		(width 1)
+		(layer "B.Cu")
+		(net 8)
+	)
+	(segment
 		(start 163.62 73)
 		(end 165.121 71.499)
@@
 	)
 	(segment
+		(start 138.5 71.499)
+		(end 138.62 71.619)
+		(width 1)
+		(layer "B.Cu")
+		(net 8)
+	)
+	(segment
 		(start 110.5 79.5)
 		(end 107.5 76.5)
@@
 	)
 	(segment
+		(start 163.62 71.619)
+		(end 163.62 73)
+		(width 1)
+		(layer "B.Cu")
+		(net 8)
+	)
+	(segment
+		(start 138.5 71.499)
+		(end 140.121 71.499)
+		(width 1)
+		(layer "B.Cu")
+		(net 8)
+	)
+	(segment
 		(start 90.121 71.499)
 		(end 112.119 71.499)
@@
 	)
 	(segment
+		(start 163.5 71.499)
+		(end 165.121 71.499)
+		(width 1)
+		(layer "B.Cu")
+		(net 8)
+	)
+	(segment
+		(start 113.5 71.499)
+		(end 115.121 71.499)
+		(width 1)
+		(layer "B.Cu")
+		(net 8)
+	)
+	(segment
 		(start 110 90)
 		(end 110.000392 90.000392)
@@
 	)
 	(segment
+		(start 162.119 71.499)
+		(end 163.5 71.499)
+		(width 1)
+		(layer "B.Cu")
+		(net 8)
+	)
+	(segment
+		(start 138.62 71.619)
+		(end 138.62 73)
+		(width 1)
+		(layer "B.Cu")
+		(net 8)
+	)
+	(segment
+		(start 113.62 73)
+		(end 113.62 71.619)
+		(width 1)
+		(layer "B.Cu")
+		(net 8)
+	)
+	(segment
 		(start 187.119 71.499)
 		(end 188.62 73)
 		(width 1)
 		(layer "B.Cu")
+		(net 8)
+	)
+	(segment
+		(start 112.119 71.499)
+		(end 113.5 71.499)
+		(width 1)
+		(layer "B.Cu")
+		(net 8)
+	)
+	(segment
+		(start 137.119 71.499)
+		(end 138.5 71.499)
+		(width 1)
+		(layer "B.Cu")
